File: Blokkendoos_binnenverlichting.kicad_sch (KiCad schematic)
At the start: 89 parts, among them J1 Conn_01x02, J10 Conn_01x04, J11 Conn_01x04, J12 Conn_01x04, J13 Conn_01x04, J2 Conn_02x11_Counter_Clockwise, J3 Conn_01x04, J4 Conn_01x02, J5 Conn_01x04, J6 Conn_01x02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

Commit message: Fixed all milestone 1 issues to date
Parts:
- added D1, D2: LED, Pyth:MHT151CYCT, symbol Device:LED
- added J14, J15: Conn_01x04, TestPoint:TestPoint_Pad_1.0x1.0mm, symbol Connector_Generic:Conn_01x01
- added Q1: 21mtc-rescue_FDC6303N-mosfet_smd, Package_TO_SOT_SMD:SOT-363_SC-70-6_Handsoldering, symbol 21mtc-cache:21mtc-rescue_FDC6303N-mosfet_smd
- added R7, R9: R, Resistor_SMD:R_0805_2012Metric_Pad1.20x1.40mm_HandSolder, symbol Device:R
- D39, D41, D43, D45: value LED -> LS A67K; footprint Pyth:MHT151CYCT -> Pyth:LED_Osram_LY_A64K; symbol Device:LED -> pyth:LED_LS_A67K; LCSC (none) -> C2830540; MFN (none) -> Osram; MPN (none) -> LS A67K-J1L2-1-0-2-R33-Z; Reichelt (none) -> G20-344
- D40, D44: value LED -> LY A67K; footprint Pyth:MHT151CYCT -> Pyth:LED_Osram_LY_A64K; symbol Device:LED -> pyth:LY A67K; LCSC (none) -> C2900136; MFN (none) -> Osram; MPN (none) -> LY A67K-J2M1-26-0-2-R33-Z; Reichelt (none) -> K04-022
- J2: LCSC (none) -> C920913; MFN (none) -> Wcon; MFP (none) -> 1310-1211G0M055CR02
Connections:
- net Aux2: now also D1.1 (K); no longer D3.1 (K)
- net Aux3: now also D2.1 (K); no longer D6.1 (K)
- net F0f: no longer D44.1 (K)
- net F0r: no longer D45.1 (K)
- net Aux5: now reaches J2.17 (Pin_17)
- net Aux5: now also Q1.1 (G), R7.1
- net GND: now reaches J2.20 (Pin_20)
- net GND: now also Q1.2 (S), Q1.5 (S), R7.2, R9.2
- net Aux6: now reaches J2.3 (Pin_3)
- net Aux6: now also Q1.3 (G), R9.1
- new net: D1.2 (A), D3.1 (K)
- new net: D2.2 (A), D6.1 (K)
- new net Aux5p: D44.1 (K), J14.1 (Pin_1), Q1.6 (D)
- new net Aux6p: D45.1 (K), J15.1 (Pin_1), Q1.4 (D)
- no-connect marks 9 -> 6
Other:
- moved on the sheet: D41, D44

Commit message: Added powerpack schematic
Other:
- added sheet PowerPack (powerpack.kicad_sch)

Commit message: Replaced FDC6303 with US6K1 in schematic
Parts:
- Q1: value 21mtc-rescue_FDC6303N-mosfet_smd -> US6K1; footprint Package_TO_SOT_SMD:SOT-363_SC-70-6_Handsoldering -> SOT-363; symbol 21mtc-cache:21mtc-rescue_FDC6303N-mosfet_smd -> pyth:US6K1; LCSC2 C83571 -> C703686; MFN FDC6303N -> US6K1; MFP Onsemi -> ROHM
- Q1: value 21mtc-rescue_FDC6303N-mosfet_smd -> US6K1; footprint Package_TO_SOT_SMD:SOT-363_SC-70-6_Handsoldering -> SOT-363; symbol 21mtc-cache:21mtc-rescue_FDC6303N-mosfet_smd -> pyth:US6K1
Connections:
- net Aux5: now also Q1.2 (G); no longer Q1.1 (G)
- net Aux6: now also Q1.5 (G); no longer Q1.3 (G)
- net Aux6p: now also Q1.3 (D); no longer Q1.4 (D)
- net GND: now also Q1.1 (S), Q1.4 (S); no longer Q1.2 (S), Q1.5 (S)
Other:
- sheet PowerPack ports: added Powerpack enable; removed none

Commit message: Removed powerpack hardware, should be on separate PCB. Replaced FDC6303, closes #12
Parts:
- Q1: footprint SOT-363 -> Package_TO_SOT_SMD:SOT-363_SC-70-6_Handsoldering
Other:
- removed sheet PowerPack

Commit message: Added motor spring mount pads, closes #9
Parts:
- added J16: Conn_01x02, Pyth:Blokkendoos motor spings, symbol Connector_Generic:Conn_01x02
Connections:
- net Motor1: now also J16.1 (Pin_1)
- net Motor2: now also J16.2 (Pin_2)
Changed lines of the file:
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@@
+    (stroke (width 0) (type default) (color 0 0 0 0))
+  )
+  (wire (pts (xy 172.72 86.995) (xy 184.15 86.995))
     (stroke (width 0) (type default) (color 0 0 0 0))
   )
@@
     (stroke (width 0) (type default) (color 0 0 0 0))
   )
+  (wire (pts (xy 172.72 84.455) (xy 184.15 84.455))
+    (stroke (width 0) (type default) (color 0 0 0 0))
+  )
   (wire (pts (xy 107.95 55.88) (xy 100.33 55.88))
     (stroke (width 0) (type default) (color 0 0 0 0))
@@
     (effects (font (size 1.27 1.27)) (justify left bottom))
   )
+  (label "Motor1" (at 172.72 84.455 0)
+    (effects (font (size 1.27 1.27)) (justify left bottom))
+  )
   (label "Aux5p" (at 48.26 179.07 0)
     (effects (font (size 1.27 1.27)) (justify left bottom))
   )
   (label "Motor2" (at 153.67 100.33 0)
+    (effects (font (size 1.27 1.27)) (justify left bottom))
+  )
+  (label "Motor2" (at 172.72 86.995 0)
     (effects (font (size 1.27 1.27)) (justify left bottom))
   )
@@
     )
     (property "Datasheet" "~" (id 3) (at 100.33 38.1 0)
+      (effects (font (size 1.27 1.27)) hide)
+    )
+    (pin "1")
+    (pin "2")
+  )
+  (symbol (lib_id "Connector_Generic:Conn_01x02") (at 189.23 84.455 0) (unit 1)
+    (in_bom yes) (on_board yes) (fields_autoplaced)
+    (property "Reference" "J16" (id 0) (at 191.262 84.8165 0)
+      (effects (font (size 1.27 1.27)) (justify left))
+    )
+    (property "Value" "Conn_01x02" (id 1) (at 191.262 87.5916 0)
+      (effects (font (size 1.27 1.27)) (justify left))
+    )
+    (property "Footprint" "Pyth:Blokkendoos motor spings" (id 2) (at 189.23 84.455 0)
+      (effects (font (size 1.27 1.27)) hide)
+    )
+    (property "Datasheet" "~" (id 3) (at 189.23 84.455 0)
       (effects (font (size 1.27 1.27)) hide)
     )
@@
       (reference "J15") (unit 1) (value "Conn_01x04") (footprint "TestPoint:TestPoint_Pad_1.0x1.0mm")
     )
+    (path "/14f07383-e637-4c44-84c4-54ea90d99c99"
+      (reference "J16") (unit 1) (value "Conn_01x02") (footprint "Pyth:Blokkendoos motor spings")
+    )
     (path "/9a6a1876-1d52-4f26-8e1b-00aa89b4c157"

Commit message: Added connectors for powerpack and DRC passes, except for silkscreen
Parts:
- added J17: Conn_01x03_Female, Connector_PinHeader_2.54mm:PinHeader_1x03_P2.54mm_Horizontal, symbol Connector:Conn_01x03_Female
- added J18: Conn_01x01, Connector_PinHeader_2.54mm:PinHeader_1x01_P2.54mm_Horizontal, symbol Connector_Generic:Conn_01x01
Connections:
- net GND: now also J17.2 (Pin_2)
- net VPP: now also J17.1 (Pin_1)
- new net Charge: J17.3 (Pin_3), J18.1 (Pin_1)
Changed lines of the file:
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@@
   (junction (at 76.2 55.88) (diameter 0) (color 0 0 0 0)
   )
+  (junction (at 182.245 76.2) (diameter 0) (color 0 0 0 0)
+  )
   (junction (at 229.87 110.49) (diameter 0) (color 0 0 0 0)
   )
@@
     (stroke (width 0) (type default) (color 0 0 0 0))
   )
+  (wire (pts (xy 173.99 73.66) (xy 182.88 73.66))
+    (stroke (width 0) (type default) (color 0 0 0 0))
+  )
   (wire (pts (xy 181.61 95.25) (xy 181.61 100.33))
     (stroke (width 0) (type default) (color 0 0 0 0))
@@
     (stroke (width 0) (type default) (color 0 0 0 0))
   )
+  (wire (pts (xy 182.88 71.12) (xy 179.07 71.12))
+    (stroke (width 0) (type default) (color 0 0 0 0))
+  )
   (wire (pts (xy 87.63 128.27) (xy 87.63 133.35))
     (stroke (width 0) (type default) (color 0 0 0 0))
@@
     (stroke (width 0) (type default) (color 0 0 0 0))
   )
+  (wire (pts (xy 173.99 77.47) (xy 173.99 73.66))
+    (stroke (width 0) (type default) (color 0 0 0 0))
+  )
   (wire (pts (xy 44.45 148.59) (xy 44.45 152.4))
     (stroke (width 0) (type default) (color 0 0 0 0))
@@
     (stroke (width 0) (type default) (color 0 0 0 0))
   )
+  (wire (pts (xy 182.245 62.865) (xy 182.245 76.2))
+    (stroke (width 0) (type default) (color 0 0 0 0))
+  )
   (wire (pts (xy 87.63 128.27) (xy 158.75 128.27))
     (stroke (width 0) (type default) (color 0 0 0 0))
@@
     (stroke (width 0) (type default) (color 0 0 0 0))
   )
+  (wire (pts (xy 175.26 76.2) (xy 182.245 76.2))
+    (stroke (width 0) (type default) (color 0 0 0 0))
+  )
   (wire (pts (xy 17.78 54.61) (xy 13.97 54.61))
     (stroke (width 0) (type default) (color 0 0 0 0))
@@
     (stroke (width 0) (type default) (color 0 0 0 0))
   )
+  (wire (pts (xy 182.245 76.2) (xy 182.88 76.2))
+    (stroke (width 0) (type default) (color 0 0 0 0))
+  )
   (wire (pts (xy 151.13 90.17) (xy 172.72 90.17))
     (stroke (width 0) (type default) (color 0 0 0 0))
@@
     (stroke (width 0) (type default) (color 0 0 0 0))
   )
+  (wire (pts (xy 184.15 62.865) (xy 182.245 62.865))
+    (stroke (width 0) (type default) (color 0 0 0 0))
+  )
   (wire (pts (xy 83.82 41.91) (xy 83.82 43.18))
     (stroke (width 0) (type default) (color 0 0 0 0))
@@
     (stroke (width 0) (type default) (color 0 0 0 0))
   )
+  (wire (pts (xy 179.07 71.12) (xy 179.07 69.85))
+    (stroke (width 0) (type default) (color 0 0 0 0))
+  )
   (text "Sluitlicht" (at 76.2 161.29 0)
     (effects (font (size 1.27 1.27)) (justify left bottom))
@@
     (effects (font (size 1.27 1.27)) (justify left bottom))
   )
+  (label "Charge" (at 175.26 76.2 0)
+    (effects (font (size 1.27 1.27)) (justify left bottom))
+  )
   (label "Aux5" (at 152.4 102.87 0)
     (effects (font (size 1.27 1.27)) (justify left bottom))
@@
     (pin "2")
   )
+  (symbol (lib_id "power:VPP") (at 179.07 69.85 0) (unit 1)
+    (in_bom yes) (on_board yes) (fields_autoplaced)
+    (property "Reference" "#PWR?" (id 0) (at 179.07 73.66 0)
+      (effects (font (size 1.27 1.27)) hide)
+    )
+    (property "Value" "VPP" (id 1) (at 179.07 66.04 0))
+    (property "Footprint" "" (id 2) (at 179.07 69.85 0)
+      (effects (font (size 1.27 1.27)) hide)
+    )
+    (property "Datasheet" "" (id 3) (at 179.07 69.85 0)
+      (effects (font (size 1.27 1.27)) hide)
+    )
+    (pin "1")
+  )
   (symbol (lib_id "Device:LED") (at 17.78 48.26 90) (unit 1)
     (in_bom yes) (on_board yes) (fields_autoplaced)
@@
     (pin "2")
   )
+  (symbol (lib_id "power:GND") (at 173.99 77.47 0) (unit 1)
+    (in_bom yes) (on_board yes) (fields_autoplaced)
+    (property "Reference" "#PWR?" (id 0) (at 173.99 83.82 0)
+      (effects (font (size 1.27 1.27)) hide)
+    )
+    (property "Value" "GND" (id 1) (at 173.99 82.0325 0))
+    (property "Footprint" "" (id 2) (at 173.99 77.47 0)
+      (effects (font (size 1.27 1.27)) hide)
+    )
+    (property "Datasheet" "" (id 3) (at 173.99 77.47 0)
+      (effects (font (size 1.27 1.27)) hide)
+    )
+    (pin "1")
+  )
   (symbol (lib_id "Connector_Generic:Conn_01x01") (at 72.39 138.43 180) (unit 1)
     (in_bom yes) (on_board yes)
@@
     (pin "2")
   )
+  (symbol (lib_id "Connector_Generic:Conn_01x01") (at 189.23 62.865 0) (unit 1)
+    (in_bom yes) (on_board yes) (fields_autoplaced)
+    (property "Reference" "J18" (id 0) (at 191.262 61.9565 0)
+      (effects (font (size 1.27 1.27)) (justify left))
+    )
+    (property "Value" "Conn_01x01" (id 1) (at 191.262 64.7316 0)
+      (effects (font (size 1.27 1.27)) (justify left))
+    )
+    (property "Footprint" "Connector_PinHeader_2.54mm:PinHeader_1x01_P2.54mm_Horizontal" (id 2) (at 189.23 62.865 0)
+      (effects (font (size 1.27 1.27)) hide)
+    )
+    (property "Datasheet" "~" (id 3) (at 189.23 62.865 0)
+      (effects (font (size 1.27 1.27)) hide)
+    )
+    (pin "1")
+  )
   (symbol (lib_id "Device:LED") (at 161.29 48.26 90) (unit 1)
     (in_bom yes) (on_board yes) (fields_autoplaced)
@@
     (pin "2")
   )
+  (symbol (lib_id "Connector:Conn_01x03_Female") (at 187.96 73.66 0) (unit 1)
+    (in_bom yes) (on_board yes) (fields_autoplaced)
+    (property "Reference" "J17" (id 0) (at 188.6712 72.7515 0)
+      (effects (font (size 1.27 1.27)) (justify left))
+    )
+    (property "Value" "Conn_01x03_Female" (id 1) (at 188.6712 75.5266 0)
+      (effects (font (size 1.27 1.27)) (justify left))
+    )
+    (property "Footprint" "Connector_PinHeader_2.54mm:PinHeader_1x03_P2.54mm_Horizontal" (id 2) (at 187.96 73.66 0)
+      (effects (font (size 1.27 1.27)) hide)
+    )
+    (property "Datasheet" "~" (id 3) (at 187.96 73.66 0)
+      (effects (font (size 1.27 1.27)) hide)
+    )
+    (pin "1")
+    (pin "2")
+    (pin "3")
+  )
   (symbol (lib_id "pyth:LY A67K") (at 48.26 171.45 90) (unit 1)
     (in_bom yes) (on_board yes)
@@
       (reference "#PWR0106") (unit 1) (value "VPP") (footprint "")
     )
+    (path "/3c55d0c6-e74c-47a0-9def-e0f177d7196e"
+      (reference "#PWR?") (unit 1) (value "VPP") (footprint "")
+    )
+    (path "/44c0ff2a-ddaa-453e-945a-0d3d31e07a29"
+      (reference "#PWR?") (unit 1) (value "GND") (footprint "")
+    )
     (path "/ad2ea191-4b92-4f8d-a2d7-0383f4505cbb"
       (reference "D1") (unit 1) (value "LED") (footprint "Pyth:MHT151CYCT")
@@
       (reference "J16") (unit 1) (value "Conn_01x02") (footprint "Pyth:Blokkendoos motor spings")
     )
+    (path "/eab04e5f-6d85-4419-bfd3-a10e4d5a8e4e"
+      (reference "J17") (unit 1) (value "Conn_01x03_Female") (footprint "Connector_PinHeader_2.54mm:PinHeader_1x03_P2.54mm_Horizontal")
+    )
+    (path "/7006d12a-53b0-4abc-aeb2-2e6eaf1d7805"
+      (reference "J18") (unit 1) (value "Conn_01x01") (footprint "Connector_PinHeader_2.54mm:PinHeader_1x01_P2.54mm_Horizontal")
+    )
     (path "/9a6a1876-1d52-4f26-8e1b-00aa89b4c157"
